Commit message: Imported upstream version '0.2.0' of 'upstream'

File: description/urdf/svh.urdf.xacro (robot description, xacro)
@@ -6,5 +6,5 @@
     <!-- BASE_LINE LINKS -->
     <joint name="${name}_base_joint" type="fixed" >
-      <insert_block name="origin" />
+      <xacro:insert_block name="origin" />
       <parent link="${parent}" />
       <child link="${name}_base_link" />
@@ -18,14 +18,20 @@
 	</geometry>
       </visual>
-    </link>
-    <link name="d">
+      <collision>
+	<origin xyz="0 0 -0.032" rpy="0 0 0" />
+	<geometry>
+          <mesh filename="package://schunk_svh_driver/description/meshes/base10.dae" />
+	</geometry>
+      </collision>
+    </link>
+    <link name="${name}_d">
       <!-- <visual> -->
       <!-- 	<geometry> -->
       <!-- 	  <cylinder length="0.110" radius="${cyl_radius}" /> -->
       <!-- 	</geometry> -->
-      <!-- 	<material name="green" /> -->
+      <!-- 	<material name="${name}_green" /> -->
       <!-- </visual> -->
     </link>
-    <link name="h">
+    <link name="${name}_h">
       <!-- <visual> -->
       <!-- 	<origin rpy="0 1.571 0" xyz="${side*(-0.0125)} 0 0.0825" /> -->
@@ -33,8 +39,8 @@
       <!-- 	  <cylinder length="0.025" radius="${cyl_radius}" /> -->
       <!-- 	</geometry> -->
-      <!-- 	<material name="green" /> -->
+      <!-- 	<material name="${name}_green" /> -->
       <!-- </visual> -->
     </link>
-    <link name="d2">
+    <link name="${name}_d2">
       <!-- <visual> -->
       <!-- 	<origin rpy="0 0 0" xyz="${side*(-0.025)} 0 0.09625" /> -->
@@ -42,9 +48,9 @@
       <!-- 	  <cylinder length="0.0275" radius="${cyl_radius}" /> -->
       <!-- 	</geometry> -->
-      <!-- 	<material name="green" /> -->
+      <!-- 	<material name="${name}_green" /> -->
       <!-- </visual> -->
     </link>
     <!-- LENGTH NOT FOUND IN DATASHEET! GUESSED!!! -->
-    <link name="e1">
+    <link name="${name}_e1">
       <visual>
 	<origin rpy="0 0 0" xyz="0 0.01313 0" />
@@ -53,7 +59,13 @@
 	</geometry>
       </visual>
+      <collision>
+	<origin rpy="0 0 0" xyz="0 0.01313 0" />
+	<geometry>
+          <mesh scale="${side*(1)} 1 1" filename="package://schunk_svh_driver/description/meshes/h10.dae" />
+	</geometry>
+      </collision>
     </link>
     <!-- LENGTH NOT FOUND IN DATASHEET! GUESSED!!! -->
-    <link name="e2">
+    <link name="${name}_e2">
       <visual>
 	<origin xyz="${side*(-0.0007)} 0 -0.01002" />
@@ -62,7 +74,13 @@
 	</geometry>
       </visual>
+      <collision>
+	<origin xyz="${side*(-0.0007)} 0 -0.01002" />
+	<geometry>
+          <mesh scale="${side*(1)} 1 1" filename="package://schunk_svh_driver/description/meshes/h11.dae" />
+	</geometry>
+      </collision>
     </link>
     <!-- LENGTH NOT FOUND IN DATASHEET! GUESSED!!! -->
-    <link name="e3">
+    <link name="${name}_e3">
       <!-- <visual> -->
       <!-- 	<origin rpy="0 0 0" xyz="${side*(0.0175)} 0 0.015" /> -->
@@ -73,8 +91,8 @@
       <!-- </visual> -->
     </link>
-    <link name="e">
+    <link name="${name}_e">
     </link>
     <!-- LENGTH NOT FOUND IN DATASHEET! GUESSED, BUT POSITION CALCULATED: E4 = D-G-F!!! -->
-    <link name="e4">
+    <link name="${name}_e4">
       <!-- <visual> -->
       <!-- 	<origin rpy="0 0 0" xyz="${side*(0.02825)} 0 0.043" /> -->
@@ -86,5 +104,5 @@
     </link>
     <!-- LENGTH NOT FOUND IN DATASHEET! GUESSED, BUT POSITION CALCULATED: E5 = D-G!!! -->
-    <link name="e5">
+    <link name="${name}_e5">
       <!-- <visual> -->
       <!-- 	<origin rpy="0 0 0" xyz="${side*(0.00675)} 0 0.04775" /> -->
@@ -96,5 +114,5 @@
     </link>
     <!-- THUMB LINKS -->
-    <link name="z">
+    <link name="${name}_z">
       <visual>
 	<origin xyz="0 0 0.02442" />
@@ -103,7 +121,13 @@
 	</geometry>
       </visual>
-    </link>
-    <link name="virtual_a" />
-    <link name="a">
+      <collision>
+	<origin xyz="0 0 0.02442" />
+	<geometry>
+          <mesh scale="1 ${side*(1)} 1" filename="package://schunk_svh_driver/description/meshes/d10.dae" />
+	</geometry>
+      </collision>
+    </link>
+    <link name="${name}_virtual_a" />
+    <link name="${name}_a">
       <visual>
 	<geometry>
@@ -111,6 +135,11 @@
 	</geometry>
       </visual>
-    </link>
-    <link name="b">
+      <collision>
+	<geometry>
+          <mesh scale="1 ${side*(1)} ${side*(1)}" filename="package://schunk_svh_driver/description/meshes/d11.dae" />
+	</geometry>
+      </collision>
+    </link>
+    <link name="${name}_b">
       <visual>
 	<geometry>
@@ -118,6 +147,11 @@
 	</geometry>
       </visual>
-    </link>
-    <link name="c">
+      <collision>
+	<geometry>
+          <mesh scale="1 ${side*(1)} ${side*(1)}" filename="package://schunk_svh_driver/description/meshes/d12.dae" />
+	</geometry>
+      </collision>
+    </link>
+    <link name="${name}_c">
       <visual>
 	<geometry>
@@ -125,7 +159,12 @@
 	</geometry>
       </visual>
+      <collision>
+	<geometry>
+          <mesh scale="1 ${side*(1)} ${side*(1)}" filename="package://schunk_svh_driver/description/meshes/d13.dae" />
+	</geometry>
+      </collision>
     </link>
     <!-- INDEX FINGER LINKS -->
-    <link name="virtual_l">
+    <link name="${name}_virtual_l">
       <visual>
 	<origin xyz="0 0 0.01321" />
@@ -134,6 +173,12 @@
 	</geometry>
       </visual>
-    </link>
-    <link name="l">
+      <collision>
+	<origin xyz="0 0 0.01321" />
+	<geometry>
+          <mesh filename="package://schunk_svh_driver/description/meshes/f10.dae" />
+	</geometry>
+      </collision>
+    </link>
+    <link name="${name}_l">
       <visual>
 	<geometry>
@@ -141,6 +186,11 @@
 	</geometry>
       </visual>
-    </link>
-    <link name="p">
+      <collision>
+	<geometry>
+          <mesh filename="package://schunk_svh_driver/description/meshes/f11.dae" />
+	</geometry>
+      </collision>
+    </link>
+    <link name="${name}_p">
       <visual>
 	<geometry>
@@ -148,6 +198,11 @@
 	</geometry>
       </visual>
-    </link>
-    <link name="t">
+      <collision>
+	<geometry>
+          <mesh filename="package://schunk_svh_driver/description/meshes/f12.dae" />
+	</geometry>
+      </collision>
+    </link>
+    <link name="${name}_t">
       <visual>
 	<geometry>
@@ -155,7 +210,12 @@
 	</geometry>
       </visual>
+      <collision>
+	<geometry>
+          <mesh filename="package://schunk_svh_driver/description/meshes/f13.dae" />
+	</geometry>
+      </collision>
     </link>
     <!-- MIDDLE FINGER LINKS -->
-    <link name="virtual_k">
+    <link name="${name}_virtual_k">
       <visual>
 	<origin xyz="0 0 0.01321" />
@@ -164,6 +224,12 @@
 	</geometry>
       </visual>
-    </link>
-    <link name="k">
+      <collision>
+	<origin xyz="0 0 0.01321" />
+	<geometry>
+          <mesh filename="package://schunk_svh_driver/description/meshes/f20.dae" />
+	</geometry>
+      </collision>
+    </link>
+    <link name="${name}_k">
       <visual>
 	<geometry>
@@ -171,6 +237,11 @@
 	</geometry>
       </visual>
-    </link>
-    <link name="o">
+      <collision>
+	<geometry>
+          <mesh filename="package://schunk_svh_driver/description/meshes/f21.dae" />
+	</geometry>
+      </collision>
+    </link>
+    <link name="${name}_o">
       <visual>
 	<geometry>
@@ -178,6 +249,11 @@
 	</geometry>
       </visual>
-    </link>
-    <link name="s">
+      <collision>
+	<geometry>
+          <mesh filename="package://schunk_svh_driver/description/meshes/f22.dae" />
+	</geometry>
+      </collision>
+    </link>
+    <link name="${name}_s">
       <visual>
 	<geometry>
@@ -185,7 +261,12 @@
 	</geometry>
       </visual>
+      <collision>
+	<geometry>
+          <mesh filename="package://schunk_svh_driver/description/meshes/f23.dae" />
+	</geometry>
+      </collision>
     </link>
     <!-- RING FINGER LINKS -->
-    <link name="virtual_j">
+    <link name="${name}_virtual_j">
       <visual>
 	<origin xyz="0 0 -0.01321" />
@@ -194,6 +275,12 @@
 	</geometry>
       </visual>
-    </link>
-    <link name="j">
+      <collision>
+	<origin xyz="0 0 -0.01321" />
+	<geometry>
+          <mesh filename="package://schunk_svh_driver/description/meshes/f30.dae" />
+	</geometry>
+      </collision>
+    </link>
+    <link name="${name}_j">
       <visual>
 	<geometry>
@@ -201,6 +288,11 @@
 	</geometry>
       </visual>
-    </link>
-    <link name="n">
+      <collision>
+	<geometry>
+          <mesh filename="package://schunk_svh_driver/description/meshes/f31.dae" />
+	</geometry>
+      </collision>
+    </link>
+    <link name="${name}_n">
       <visual>
 	<geometry>
@@ -208,6 +300,11 @@
 	</geometry>
       </visual>
-    </link>
-    <link name="r">
+      <collision>
+	<geometry>
+          <mesh filename="package://schunk_svh_driver/description/meshes/f32.dae" />
+	</geometry>
+      </collision>
+    </link>
+    <link name="${name}_r">
       <visual>
 	<geometry>
@@ -215,7 +312,12 @@
 	</geometry>
       </visual>
+      <collision>
+	<geometry>
+          <mesh filename="package://schunk_svh_driver/description/meshes/f33.dae" />
+	</geometry>
+      </collision>
     </link>
     <!-- LITTLE FINGER LINKS -->
-    <link name="virtual_i">
+    <link name="${name}_virtual_i">
       <visual>
 	<origin xyz="0 0 -0.01321" />
@@ -224,6 +326,12 @@
 	</geometry>
       </visual>
-    </link>
-    <link name="i">
+      <collision>
+	<origin xyz="0 0 -0.01321" />
+	<geometry>
+          <mesh filename="package://schunk_svh_driver/description/meshes/f40.dae" />
+	</geometry>
+      </collision>
+    </link>
+    <link name="${name}_i">
       <visual>
 	<geometry>
@@ -231,6 +339,11 @@
 	</geometry>
       </visual>
-    </link>
-    <link name="m">
+      <collision>
+	<geometry>
+          <mesh filename="package://schunk_svh_driver/description/meshes/f41.dae" />
+	</geometry>
+      </collision>
+    </link>
+    <link name="${name}_m">
       <visual>
 	<geometry>
@@ -238,6 +351,11 @@
 	</geometry>
       </visual>
-    </link>
-    <link name="q">
+      <collision>
+	<geometry>
+          <mesh filename="package://schunk_svh_driver/description/meshes/f42.dae" />
+	</geometry>
+      </collision>
+    </link>
+    <link name="${name}_q">
       <visual>
 	<geometry>
@@ -245,21 +363,26 @@
 	</geometry>
       </visual>
-    </link>
-    <joint name="Thumb_Flexion" type="revolute">
-      <parent link="virtual_a" />
-      <child link="a" />
+      <collision>
+	<geometry>
+          <mesh filename="package://schunk_svh_driver/description/meshes/f43.dae" />
+	</geometry>
+      </collision>
+    </link>
+    <joint name="${name}_Thumb_Flexion" type="revolute">
+      <parent link="${name}_virtual_a" />
+      <child link="${name}_a" />
       <limit effort="1000.0" lower="0.0" upper="0.9704" velocity="1" />
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